Commit message: URDF Updates

File: src/Simulation/urdf/hapticdevice_URDF.urdf (robot description, URDF)
Before this commit: robot hapticdevice_URDF, 9 links, 8 joints
Links:
- link base_link: geometry collision mesh filename=package://haptic_sim/meshes/base_link.STL; visual mesh filename=package://haptic_sim/meshes/base_link.STL
- link link1: geometry collision mesh filename=package://haptic_sim/meshes/link1.STL; visual mesh filename=package://haptic_sim/meshes/link1.STL
- link link2: geometry collision mesh filename=package://haptic_sim/meshes/link2.STL; visual mesh filename=package://haptic_sim/meshes/link2.STL
- link link3: geometry collision mesh filename=package://haptic_sim/meshes/link3.STL; visual mesh filename=package://haptic_sim/meshes/link3.STL
- link link3b: geometry collision mesh filename=package://haptic_sim/meshes/link3b.STL; visual mesh filename=package://haptic_sim/meshes/link3b.STL
- link link4: geometry collision mesh filename=package://haptic_sim/meshes/link4.STL; visual mesh filename=package://haptic_sim/meshes/link4.STL
- link link5: geometry collision mesh filename=package://haptic_sim/meshes/link5.STL; visual mesh filename=package://haptic_sim/meshes/link5.STL
- link link6: geometry collision mesh filename=package://haptic_sim/meshes/link6.STL; visual mesh filename=package://haptic_sim/meshes/link6.STL
